File: power-module/power-module.kicad_pcb (KiCad board)
At the start: 2 copper layers, 74.9 x 27.9 mm, 20 parts, among them J1 Barrel_Jack, J3 Conn_01x03_Pin, SW1 SW_Push, SW2 SW_SPST, SW3 SW_SPDT, U1 L7805, U2 NE555P, U3 NE555P

Commit message: add some thingies
Parts:
- moved J1 0.63 mm to (129.9, 57.1)
Other:
- board text added: "JLCJLCJLCJLC"
Changed lines of the file:
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@@
   )
   (footprint "Connector_BarrelJack:BarrelJack_SwitchcraftConxall_RAPC10U_Horizontal" (layer "F.Cu")
-    (at 129.28 57.15)
+    (at 129.915 57.15)
     (descr "DC Power Jack, 13A, 24V, Panel Mount,Through-hole, https://www.switchcraft.com/Drawings/RAPC10U_CD.pdf")
     (tags "barreljack switchcraftconxall dc power")
@@
     (property "ki_keywords" "R res resistor")
     (attr through_hole)
-    (fp_text reference "R5" (at 5.08 -2.37) (layer "F.SilkS")
+    (fp_text reference "R5" (at 5.08 -2.37) (layer "F.SilkS") hide
         (effects (font (size 1 1) (thickness 0.15)))
     )
@@
   (gr_rect (start 111.125 43.18) (end 186.055 71.12)
     (stroke (width 0.1) (type default)) (fill none) (layer "Edge.Cuts"))
+  (gr_text "JLCJLCJLCJLC" (at 112.5 57.5) (layer "F.SilkS")
+    (effects (font (size 1 1) (thickness 0.15)) (justify left bottom))
+  )
   (segment (start 127.635 46.99) (end 123.2325 46.99) (width 0.25) (layer "F.Cu") (net 1))
   (segment (start 128.27 47.625) (end 127.635 46.99) (width 0.25) (layer "F.Cu") (net 1))
   (via (at 128.27 47.625) (size 0.8) (drill 0.4) (layers "F.Cu" "B.Cu") (net 1))
-  (segment (start 129.28 57.15) (end 129.28 48.635) (width 0.25) (layer "B.Cu") (net 1))
-  (segment (start 129.28 48.635) (end 128.27 47.625) (width 0.25) (layer "B.Cu") (net 1))
+  (segment (start 129.915 49.27) (end 129.915 57.15) (width 0.25) (layer "B.Cu") (net 1))
+  (segment (start 128.27 47.625) (end 129.915 49.27) (width 0.25) (layer "B.Cu") (net 1))
   (segment (start 163.965 54.475) (end 151.61 54.475) (width 0.25) (layer "F.Cu") (net 2))
   (segment (start 151.61 54.475) (end 150.485 53.35) (width 0.25) (layer "F.Cu") (net 2))
@@
   (segment (start 149.225 66.675) (end 150.495 65.405) (width 0.25) (layer "F.Cu") (net 2))
   (segment (start 167.235 66.675) (end 168.91 66.675) (width 0.25) (layer "F.Cu") (net 2))
+  (segment (start 117.475 57.15) (end 124.735 57.15) (width 0.25) (layer "F.Cu") (net 2))
   (segment (start 150.495 65.405) (end 156.21 65.405) (width 0.25) (layer "F.Cu") (net 2))
   (segment (start 136.525 66.675) (end 135.6 65.75) (width 0.25) (layer "F.Cu") (net 2))
@@
   (segment (start 130.115 65.75) (end 131.04 66.675) (width 0.25) (layer "F.Cu") (net 2))
   (segment (start 165.09 53.35) (end 163.965 54.475) (width 0.25) (layer "F.Cu") (net 2))
-  (segment (start 117.475 57.15) (end 124.1 57.15) (width 0.25) (layer "F.Cu") (net 2))
   (segment (start 163.485 67.6) (end 166.31 67.6) (width 0.25) (layer "F.Cu") (net 2))
   (segment (start 149.225 66.675) (end 147.32 66.675) (width 0.25) (layer "F.Cu") (net 2))
@@
   (segment (start 169.545 66.04) (end 169.545 64.77) (width 0.25) (layer "B.Cu") (net 2))
   (segment (start 149.225 64.77) (end 149.225 66.675) (width 0.25) (layer "B.Cu") (net 2))
+  (segment (start 125.73 66.675) (end 125.73 65.405) (width 0.25) (layer "B.Cu") (net 2))
   (segment (start 151.145 47.555) (end 151.145 52.69) (width 0.25) (layer "B.Cu") (net 2))
   (segment (start 151.145 52.69) (end 150.485 53.35) (width 0.25) (layer "B.Cu") (net 2))
   (segment (start 116.84 67.62) (end 116.84 57.785) (width 0.25) (layer "B.Cu") (net 2))
+  (segment (start 124.735 64.41) (end 124.735 57.15) (width 0.25) (layer "B.Cu") (net 2))
   (segment (start 169.545 64.77) (end 169.545 57.805) (width 0.25) (layer "B.Cu") (net 2))
-  (segment (start 125.73 58.78) (end 124.1 57.15) (width 0.25) (layer "B.Cu") (net 2))
+  (segment (start 125.73 65.405) (end 124.735 64.41) (width 0.25) (layer "B.Cu") (net 2))
   (segment (start 169.545 57.805) (end 165.09 53.35) (width 0.25) (layer "B.Cu") (net 2))
   (segment (start 149.225 54.61) (end 149.225 64.77) (width 0.25) (layer "B.Cu") (net 2))
-  (segment (start 125.73 66.675) (end 125.73 58.78) (width 0.25) (layer "B.Cu") (net 2))
   (segment (start 150.485 53.35) (end 149.225 54.61) (width 0.25) (layer "B.Cu") (net 2))
   (segment (start 116.84 57.785) (end 117.475 57.15) (width 0.25) (layer "B.Cu") (net 2))
