File: regfile/regfile.kicad_sch (KiCad schematic)
At the start: 15 parts, among them J1 Conn_01x39_Pin, U1 74LS670, U10 74LS00, U11 74LS670, U12 74LS670, U13 74LS670, U14 74LS670, U2 74LS670, U3 74LS670, U4 74LS670, U5 74LS00, U6 74LS00, U7 74LS00, U8 74LS00, U9 74LS00

Commit message: A
Parts:
- removed U10, U9: 74LS00, symbol 74xx:74LS00
- added unit 2 of U6
- added unit 1 of U6
- added unit 1 of U7
- added unit 5 of U7
- added unit 2 of U7
- added unit 5 of U8
- U1, U11, U12, U13, U14, U2, U3, U4: footprint (none) -> Package_DIP:DIP-16_W7.62mm
- U5, U6, U7, U8: footprint (none) -> Package_DIP:DIP-14_W7.62mm
Connections:
- net write enable 1 is gone; now on net write enable: U5.1, U5.9, U6.9, U7.9, U8.1, U8.9
- net +5V: now also U7.14 (VCC), U8.14 (VCC)
- net GND: now also U7.7 (GND), U8.7 (GND)
- net read enable 1: now also U6.4; no longer U7.12, U8.12, U8.4
- net read enable 2: now also U7.12, U8.12, U8.4, U7.4
- net write enable: now also U6.1, U7.1
- net at J1.9 (Pin_9), U5.10, U5.2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: now also U6.2, U7.2
- net at U8.8: now also U14.12 (~{Ew}); no longer U12.12 (~{Ew})
- net at U11.1 (D2), U13.1 (D2): now also J1.17 (Pin_17), U1.1 (D2), U3.1 (D2)
- net at U13.11 (~{Er}): now also U8.6
- net at U13.12 (~{Ew}): now also U8.3
- net at U11.15 (D1), U13.15 (D1): now also J1.16 (Pin_16), U1.15 (D1), U3.15 (D1)
- net at U11.2 (D3), U13.2 (D3): now also J1.18 (Pin_18), U1.2 (D3), U3.2 (D3)
- net at U11.3 (D4), U13.3 (D4): now also J1.19 (Pin_19), U1.3 (D4), U3.3 (D4)
- net at J1.15 (Pin_15), U8.13, U8.5: now also U7.13, U7.5
- net at U11.11 (~{Er}): now also U7.6; no longer U8.6
- net at J1.12 (Pin_12), U5.13, U5.5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: now also U6.5; no longer U7.13
- net at J1.21 (Pin_21), U2.1 (D2), U4.1 (D2): now also U12.1 (D2), U14.1 (D2)
- net at U4.11 (~{Er}): now also U6.11; no longer U7.11
- net at U4.12 (~{Ew}): now also U6.8; no longer U7.8
- net at J1.20 (Pin_20), U2.15 (D1), U4.15 (D1): now also U12.15 (D1), U14.15 (D1)
- net at J1.22 (Pin_22), U2.2 (D3), U4.2 (D3): now also U12.2 (D3), U14.2 (D3)
- net at J1.23 (Pin_23), U2.3 (D4), U4.3 (D4): now also U12.3 (D4), U14.3 (D4)
- net at U3.11 (~{Er}): now also U6.6; no longer U6.11
- net at U11.12 (~{Ew}): now also U7.3; no longer U8.3
- net at U12.11 (~{Er}): now also U7.11; no longer U8.11
- net at U3.12 (~{Ew}): now also U6.3; no longer U6.8
- net at U14.11 (~{Er}): now also U8.11
- new net: U12.12 (~{Ew}), U7.8

Commit message: dwadwdawdaw
Connections:
- net at J1.8 (Pin_8), U1.13 (Wb), U11.13 (Wb)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: now also U14.13 (Wb), U4.13 (Wb)
- net at J1.7 (Pin_7), U1.14 (Wa), U11.14 (Wa)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: no longer U14.13 (Wb), U4.13 (Wb)
Changed lines of the file:
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@@
   (junction (at 339.09 203.2) (diameter 0) (color 0 0 0 0)
   )
-  (junction (at 127 212.09) (diameter 0) (color 0 0 0 0)
-  )
   (junction (at 212.09 156.21) (diameter 0) (color 0 0 0 0)
   )
@@
   (junction (at 125.73 161.29) (diameter 0) (color 0 0 0 0)
   )
+  (junction (at 255.27 213.36) (diameter 0) (color 0 0 0 0)
+  )
   (junction (at 256.54 160.02) (diameter 0) (color 0 0 0 0)
   )
@@
   (junction (at 111.76 46.99) (diameter 0) (color 0 0 0 0)
   )
+  (junction (at 125.73 212.09) (diameter 0) (color 0 0 0 0)
+  )
   (junction (at 250.19 223.52) (diameter 0) (color 0 0 0 0)
   )
@@
   (junction (at 113.03 44.45) (diameter 0) (color 0 0 0 0)
   )
-  (junction (at 256.54 213.36) (diameter 0) (color 0 0 0 0)
-  )
   (junction (at 124.46 219.71) (diameter 0) (color 0 0 0 0)
   )
@@
     (stroke (width 0) (type default))
   )
+  (wire (pts (xy 255.27 213.36) (xy 255.27 242.57))
+    (stroke (width 0) (type default))
+  )
   (wire (pts (xy 39.37 130.81) (xy 91.44 130.81))
     (stroke (width 0) (type default))
@@
     (stroke (width 0) (type default))
   )
+  (wire (pts (xy 125.73 212.09) (xy 170.18 212.09))
+    (stroke (width 0) (type default))
+  )
   (wire (pts (xy 83.82 158.75) (xy 39.37 158.75))
     (stroke (width 0) (type default))
@@
     (stroke (width 0) (type default))
   )
+  (wire (pts (xy 299.72 213.36) (xy 255.27 213.36))
+    (stroke (width 0) (type default))
+  )
   (wire (pts (xy 175.26 212.09) (xy 171.45 212.09))
     (stroke (width 0) (type default))
@@
     (stroke (width 0) (type default))
   )
-  (wire (pts (xy 127 209.55) (xy 127 212.09))
+  (wire (pts (xy 127 209.55) (xy 127 241.3))
     (stroke (width 0) (type default))
   )
@@
     (stroke (width 0) (type default))
   )
-  (wire (pts (xy 256.54 210.82) (xy 256.54 213.36))
+  (wire (pts (xy 256.54 210.82) (xy 256.54 242.57))
     (stroke (width 0) (type default))
   )
@@
     (stroke (width 0) (type default))
   )
-  (wire (pts (xy 125.73 161.29) (xy 125.73 241.3))
+  (wire (pts (xy 125.73 161.29) (xy 125.73 212.09))
+    (stroke (width 0) (type default))
+  )
+  (wire (pts (xy 125.73 212.09) (xy 125.73 241.3))
     (stroke (width 0) (type default))
   )
@@
     (stroke (width 0) (type default))
   )
-  (wire (pts (xy 256.54 213.36) (xy 299.72 213.36))
-    (stroke (width 0) (type default))
-  )
   (wire (pts (xy 304.8 77.47) (xy 304.8 71.12))
     (stroke (width 0) (type default))
@@
     (stroke (width 0) (type default))
   )
-  (wire (pts (xy 127 212.09) (xy 127 241.3))
-    (stroke (width 0) (type default))
-  )
   (wire (pts (xy 302.26 167.64) (xy 304.8 167.64))
     (stroke (width 0) (type default))
@@
     (stroke (width 0) (type default))
   )
-  (wire (pts (xy 256.54 213.36) (xy 256.54 242.57))
-    (stroke (width 0) (type default))
-  )
   (wire (pts (xy 247.65 80.01) (xy 283.21 80.01))
     (stroke (width 0) (type default))
@@
     (stroke (width 0) (type default))
   )
-  (wire (pts (xy 127 212.09) (xy 170.18 212.09))
-    (stroke (width 0) (type default))
-  )
   (wire (pts (xy 175.26 237.49) (xy 175.26 227.33))
     (stroke (width 0) (type default))
@@
     (stroke (width 0) (type default))
   )
-  (wire (pts (xy 255.27 162.56) (xy 255.27 242.57))
-    (stroke (width 0) (type default))
-  )
+  (wire (pts (xy 255.27 162.56) (xy 255.27 213.36))
+    (stroke (width 0) (type default))
+  )

Commit message: fix logic for the regfile
Parts:
- removed U5, U6, U7, U8: 74LS00, Package_DIP:DIP-14_W7.62mm, symbol 74xx:74LS00
- added U16, U17: 74LS244, Package_DIP:DIP-20_W7.62mm, symbol 74xx:74LS244
- added U18: 74LS27, Package_DIP:DIP-14_W7.62mm, symbol 74xx:74LS27
- added U5, U7: 74HC00, symbol 74xx:74HC00
- added U6: 74HC04, symbol 74xx:74HC04
- added U8: 74LS32, symbol 74xx:74LS32
Connections:
- net +5V: now also U16.20 (VCC), U17.20 (VCC), U18.14 (VCC), U5.14 (VCC), U6.14 (VCC), U7.14 (VCC), U8.14 (VCC)
- net GND: now also U16.10 (GND), U16.11 (I0b), U16.13 (I1b), U16.15 (I2b), U16.17 (I3b), U16.2 (I0a), U16.4 (I1a), U16.6 (I2a), U16.8 (I3a), U17.10 (GND), U17.11 (I0b), U17.13 (I1b), U17.15 (I2b), U17.17 (I3b), U17.2 (I0a), U17.4 (I1a), U17.6 (I2a), U17.8 (I3a), U18.10, U18.11, U18.7 (GND), U18.9, U5.7 (GND), U6.11, U6.13, U6.7 (GND), U6.9, U7.10, U7.12, U7.13, U7.7 (GND), U7.9, U8.7 (GND)
- net read enable 1: now also U5.12, U5.9
- net read enable 2: now also U7.1, U7.4
- net write enable: now also U5.1, U5.4
- net at J1.15 (Pin_15): now also U18.3, U6.5, U7.5
- net read enable R bank 2: now reaches U13.11 (~{Er})
- net read enable R bank 2: now also U14.11 (~{Er}), U8.11
- net at J1.32 (Pin_32), U11.10 (Q1), U13.10 (Q1): now also U16.3 (O3b)
- net write enable bank 2: now reaches U13.12 (~{Ew})
- net write enable bank 2: now also U14.12 (~{Ew}), U3.12 (~{Ew}), U4.12 (~{Ew}), U5.6
- net at J1.14 (Pin_14), U11.4 (Rb), U12.4 (Rb)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: now also U18.4
- net at J1.13 (Pin_13), U11.5 (Ra), U12.5 (Ra)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: now also U18.5
- net at J1.35 (Pin_35), U11.6 (Q4), U13.6 (Q4): now also U16.9 (O0b)
- net at J1.34 (Pin_34), U11.7 (Q3), U13.7 (Q3): now also U16.7 (O1b)
- net at J1.33 (Pin_33), U11.9 (Q2), U13.9 (Q2): now also U16.5 (O2b)
- net read enable L bank 2: now reaches U4.11 (~{Er})
- net read enable L bank 2: now also U3.11 (~{Er}), U8.6
- net at J1.12 (Pin_12): now also U18.13, U5.10, U6.3
- net read enable L bank 1: now reaches U1.11 (~{Er})
- net read enable L bank 1: now also U2.11 (~{Er}), U8.3
- net at J1.28 (Pin_28), U2.10 (Q1), U4.10 (Q1): now also U17.12 (O3a)
- net at J1.11 (Pin_11), U1.4 (Rb), U2.4 (Rb)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: now also U18.2
- net at J1.10 (Pin_10), U1.5 (Ra), U2.5 (Ra)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: now also U18.1
- net at J1.31 (Pin_31), U2.6 (Q4), U4.6 (Q4): now also U17.18 (O0a)
- net at J1.30 (Pin_30), U2.7 (Q3), U4.7 (Q3): now also U17.16 (O1a)
- net at J1.29 (Pin_29), U2.9 (Q2), U4.9 (Q2): now also U17.14 (O2a)
- net at J1.24 (Pin_24), U1.10 (Q1), U3.10 (Q1): now also U17.3 (O3b)
- net at J1.25 (Pin_25), U1.9 (Q2), U3.9 (Q2): now also U17.5 (O2b)
- net at J1.26 (Pin_26), U1.7 (Q3), U3.7 (Q3): now also U17.7 (O1b)
- net at J1.27 (Pin_27), U1.6 (Q4), U3.6 (Q4): now also U17.9 (O0b)
- net at J1.36 (Pin_36), U12.10 (Q1), U14.10 (Q1): now also U16.12 (O3a)
- net at J1.37 (Pin_37), U12.9 (Q2), U14.9 (Q2): now also U16.14 (O2a)
- net at J1.38 (Pin_38), U12.7 (Q3), U14.7 (Q3): now also U16.16 (O1a)
- net at J1.39 (Pin_39), U12.6 (Q4), U14.6 (Q4): now also U16.18 (O0a)
- net at J1.9 (Pin_9): now also U5.2, U6.1
- net write enable bank 1: now reaches U11.12 (~{Ew})
- net write enable bank 1: now also U1.12 (~{Ew}), U12.12 (~{Ew}), U2.12 (~{Ew}), U5.3
- net read enable R bank 1: now reaches U12.11 (~{Er})
- net read enable R bank 1: now also U11.11 (~{Er}), U8.8
- new net: U7.6, U8.9
- new net: U5.5, U6.2
- new net: U7.3, U8.12
- new net: U6.6, U7.2
- new net: U5.11, U8.4
- new net: U5.13, U6.4
- new net: U5.8, U8.1
- new net ZR_addr1: U17.1 (OEa), U17.19 (OEb), U18.12, U8.2, U8.5
- new net ZR_addr2: U16.1 (OEa), U16.19 (OEb), U18.6, U8.10, U8.13
Other:
- moved on the sheet: J1, U1, U11, U12, U13, U14, U2, U3, U4
