File: regfile/regfile.kicad_sch (KiCad schematic)
At the start: 16 parts, among them J1 Conn_01x39_Pin, U1 74LS670, U11 74LS670, U12 74LS670, U13 74LS670, U14 74LS670, U16 74LS244, U17 74LS244, U18 74LS27, U2 74LS670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

Commit message: footprints
Parts:
- U5, U6, U7, U8: footprint (none) -> Package_DIP:DIP-14_W7.62mm
Changed lines of the file:
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@@
       (effects (font (size 1.27 1.27)))
     )
-    (property "Footprint" "" (at 267.97 21.59 0)
+    (property "Footprint" "Package_DIP:DIP-14_W7.62mm" (at 267.97 21.59 0)
       (effects (font (size 1.27 1.27)) hide)
     )
@@
       (effects (font (size 1.27 1.27)))
     )
-    (property "Footprint" "" (at 283.21 24.13 0)
+    (property "Footprint" "Package_DIP:DIP-14_W7.62mm" (at 283.21 24.13 0)
       (effects (font (size 1.27 1.27)) hide)
     )
@@
       (effects (font (size 1.27 1.27)))
     )
-    (property "Footprint" "" (at 142.24 41.91 0)
+    (property "Footprint" "Package_DIP:DIP-14_W7.62mm" (at 142.24 41.91 0)
       (effects (font (size 1.27 1.27)) hide)
     )
@@
       (effects (font (size 1.27 1.27)))
     )
-    (property "Footprint" "" (at 375.92 129.54 0)
+    (property "Footprint" "Package_DIP:DIP-14_W7.62mm" (at 375.92 129.54 0)
       (effects (font (size 1.27 1.27)) hide)
     )
@@
       (effects (font (size 1.27 1.27)) (justify left))
     )
-    (property "Footprint" "" (at 374.65 207.01 0)
+    (property "Footprint" "Package_DIP:DIP-14_W7.62mm" (at 374.65 207.01 0)
       (effects (font (size 1.27 1.27)) hide)
     )
@@
       (effects (font (size 1.27 1.27)))
     )
-    (property "Footprint" "" (at 283.21 43.18 0)
+    (property "Footprint" "Package_DIP:DIP-14_W7.62mm" (at 283.21 43.18 0)
       (effects (font (size 1.27 1.27)) hide)
     )
@@
       (effects (font (size 1.27 1.27)))
     )
-    (property "Footprint" "" (at 267.97 40.64 0)
+    (property "Footprint" "Package_DIP:DIP-14_W7.62mm" (at 267.97 40.64 0)
       (effects (font (size 1.27 1.27)) hide)
     )
@@
       (effects (font (size 1.27 1.27)))
     )
-    (property "Footprint" "" (at 88.9 40.64 0)
+    (property "Footprint" "Package_DIP:DIP-14_W7.62mm" (at 88.9 40.64 0)
       (effects (font (size 1.27 1.27)) hide)
     )
@@
       (effects (font (size 1.27 1.27)))
     )
-    (property "Footprint" "" (at 104.14 43.18 0)
+    (property "Footprint" "Package_DIP:DIP-14_W7.62mm" (at 104.14 43.18 0)
       (effects (font (size 1.27 1.27)) hide)
     )
@@
       (effects (font (size 1.27 1.27)))
     )
-    (property "Footprint" "" (at 104.14 25.4 0)
+    (property "Footprint" "Package_DIP:DIP-14_W7.62mm" (at 104.14 25.4 0)
       (effects (font (size 1.27 1.27)) hide)
     )
@@
       (effects (font (size 1.27 1.27)) (justify left))
     )
-    (property "Footprint" "" (at 417.83 207.01 0)
+    (property "Footprint" "Package_DIP:DIP-14_W7.62mm" (at 417.83 207.01 0)
       (effects (font (size 1.27 1.27)) hide)
     )
@@
       (effects (font (size 1.27 1.27)))
     )
-    (property "Footprint" "" (at 375.92 86.36 0)
+    (property "Footprint" "Package_DIP:DIP-14_W7.62mm" (at 375.92 86.36 0)
       (effects (font (size 1.27 1.27)) hide)
     )
@@
       (effects (font (size 1.27 1.27)))
     )
-    (property "Footprint" "" (at 73.66 43.18 0)
+    (property "Footprint" "Package_DIP:DIP-14_W7.62mm" (at 73.66 43.18 0)
       (effects (font (size 1.27 1.27)) hide)
     )
@@
       (effects (font (size 1.27 1.27)) (justify left))
     )
-    (property "Footprint" "" (at 440.69 207.01 0)
+    (property "Footprint" "Package_DIP:DIP-14_W7.62mm" (at 440.69 207.01 0)
       (effects (font (size 1.27 1.27)) hide)
     )
@@
       (effects (font (size 1.27 1.27)))
     )
-    (property "Footprint" "" (at 88.9 22.86 0)
+    (property "Footprint" "Package_DIP:DIP-14_W7.62mm" (at 88.9 22.86 0)
       (effects (font (size 1.27 1.27)) hide)
     )
@@
       (effects (font (size 1.27 1.27)))
     )
-    (property "Footprint" "" (at 157.48 25.4 0)
+    (property "Footprint" "Package_DIP:DIP-14_W7.62mm" (at 157.48 25.4 0)
       (effects (font (size 1.27 1.27)) hide)
     )
@@
       (effects (font (size 1.27 1.27)))
     )
-    (property "Footprint" "" (at 375.92 101.6 0)
+    (property "Footprint" "Package_DIP:DIP-14_W7.62mm" (at 375.92 101.6 0)
       (effects (font (size 1.27 1.27)) hide)
     )
@@
       (effects (font (size 1.27 1.27)) (justify left))
     )
-    (property "Footprint" "" (at 464.82 207.01 0)
+    (property "Footprint" "Package_DIP:DIP-14_W7.62mm" (at 464.82 207.01 0)
       (effects (font (size 1.27 1.27)) hide)
     )
@@
       (effects (font (size 1.27 1.27)))
     )
-    (property "Footprint" "" (at 157.48 39.37 0)
+    (property "Footprint" "Package_DIP:DIP-14_W7.62mm" (at 157.48 39.37 0)
       (effects (font (size 1.27 1.27)) hide)
     )
@@
       (effects (font (size 1.27 1.27)))
     )
-    (property "Footprint" "" (at 375.92 118.11 0)
+    (property "Footprint" "Package_DIP:DIP-14_W7.62mm" (at 375.92 118.11 0)
       (effects (font (size 1.27 1.27)) hide)
     )
@@
       (effects (font (size 1.27 1.27)))
     )
-    (property "Footprint" "" (at 252.73 43.18 0)
+    (property "Footprint" "Package_DIP:DIP-14_W7.62mm" (at 252.73 43.18 0)
       (effects (font (size 1.27 1.27)) hide)
     )
@@
       (effects (font (size 1.27 1.27)))
     )
-    (property "Footprint" "" (at 375.92 144.78 0)
-      (effects (font (size 1.27 1.27)) hide)
-    )
+    (property "Footprint" "Package_DIP:DIP-14_W7.62mm" (at 375.92 144.78 0)
+      (effects (font (size 1.27 1.27)) hide)
+    )

Commit message: finish regfile
Other:
- moved on the sheet: U6F
Changed lines of the file:
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@@
   (junction (at 217.17 195.58) (diameter 0) (color 0 0 0 0)
   )
-  (junction (at 368.3 144.78) (diameter 0) (color 0 0 0 0)
-  )
   (junction (at 242.57 242.57) (diameter 0) (color 0 0 0 0)
   )
@@
   (junction (at 116.84 144.78) (diameter 0) (color 0 0 0 0)
   )
+  (junction (at 368.3 143.51) (diameter 0) (color 0 0 0 0)
+  )
   (junction (at 213.36 289.56) (diameter 0) (color 0 0 0 0)
   )
@@
   (junction (at 114.3 198.12) (diameter 0) (color 0 0 0 0)
   )
-  (wire (pts (xy 368.3 129.54) (xy 368.3 144.78))
+  (wire (pts (xy 368.3 129.54) (xy 368.3 143.51))
     (stroke (width 0) (type default))
   )
@@
     (stroke (width 0) (type default))
   )
+  (wire (pts (xy 368.3 143.51) (xy 368.3 147.32))
+    (stroke (width 0) (type default))
+  )
   (wire (pts (xy 179.07 149.86) (xy 129.54 149.86))
     (stroke (width 0) (type default))
@@
     (stroke (width 0) (type default))
   )
-  (wire (pts (xy 368.3 144.78) (xy 368.3 147.32))
-    (stroke (width 0) (type default))
-  )
   (wire (pts (xy 43.18 127) (xy 68.58 127))
     (stroke (width 0) (type default))
@@
     )
   )
-  (symbol (lib_id "74xx:74HC04") (at 375.92 144.78 0) (unit 6)
+  (symbol (lib_id "74xx:74HC04") (at 375.92 143.51 0) (unit 6)
     (in_bom yes) (on_board yes) (dnp no) (fields_autoplaced)
-    (property "Reference" "U6" (at 375.92 135.89 0)
+    (property "Reference" "U6" (at 375.92 134.62 0)
       (effects (font (size 1.27 1.27)))
     )
-    (property "Value" "74HC04" (at 375.92 138.43 0)
+    (property "Value" "74HC04" (at 375.92 137.16 0)
       (effects (font (size 1.27 1.27)))
     )
-    (property "Footprint" "Package_DIP:DIP-14_W7.62mm" (at 375.92 144.78 0)
+    (property "Footprint" "Package_DIP:DIP-14_W7.62mm" (at 375.92 143.51 0)
       (effects (font (size 1.27 1.27)) hide)
     )
-    (property "Datasheet" "https://assets.nexperia.com/documents/data-sheet/74HC_HCT04.pdf" (at 375.92 144.78 0)
+    (property "Datasheet" "https://assets.nexperia.com/documents/data-sheet/74HC_HCT04.pdf" (at 375.92 143.51 0)
       (effects (font (size 1.27 1.27)) hide)
     )
